Commit message: add interfacing plate

File: urdf/i3dr_titania_kinova.urdf.xacro (robot description, xacro)
@@ -7,11 +7,13 @@
     <xacro:arg name="en_imu" default="false"/>
     <xacro:arg name="camera_name" default="i3dr_titania"/>
-    <xacro:arg name="arm_name" default="j2s7s300"/>
+    <xacro:arg name="arm_name" default="j2s7s000"/>
     <xacro:arg name="en_mesh" default="true"/>
     <xacro:include filename="$(find i3dr_titania)/urdf/titania.urdf.xacro" />
     <xacro:titania_camera camera_name="$(arg camera_name)" en_mesh="$(arg en_mesh)" en_imu="$(arg en_imu)"/>
-    <xacro:include filename="$(find kinova_description)/urdf/$(arg arm_name).xacro" />
+    <xacro:include filename="$(find i3dr_kinova)/urdf/interfacing_plate.urdf.xacro" />
+    <xacro:interfacing_plate />
+    <xacro:include filename="$(find i3dr_kinova)/urdf/$(arg arm_name).xacro" />
     <link name="root" />
-    <xacro:j2s7s300 base_parent="root"/>
+    <xacro:j2s7s000 base_parent="root"/>
     <link name="world" />
     <joint name="world_joint" type="fixed">
@@ -20,5 +22,5 @@
         <origin xyz="0 0 0.01" rpy="0 0 0" />
     </joint>
-    <link name="ground_plane_box">
+    <!--<link name="ground_plane_box">
         <visual>
             <origin xyz="0 0 0" rpy="0 0 0"/>
@@ -42,7 +44,13 @@
         <origin xyz="0 0 -0.25" rpy="0 0 0" />
     </joint>
-    <joint name="kinova_titania_joint" type="fixed">
-        <origin xyz="0 0 0.09" rpy="-1.57 0 1.57" />
+    -->
+    <joint name="kinova_interface_joint" type="fixed">
         <parent link="$(arg arm_name)_end_effector" />
+        <child link = "interfacing_plate_base_link" />
+        <origin xyz="0 0 0" rpy="0 0 0" />
+    </joint>
+    <joint name="interface_titania_joint" type="fixed">
+        <origin xyz="0 0 0" rpy="0 0 0" />
+        <parent link="interfacing_plate_camera_mount_link" />
         <child link="$(arg camera_name)_base_link" />
     </joint>

Commit message: hide gazebo world floor (robot gets stuck)

File: urdf/i3dr_titania_kinova.urdf.xacro (robot description, xacro)
@@ -10,8 +10,10 @@
     <xacro:arg name="en_mesh" default="true"/>
     <xacro:include filename="$(find i3dr_titania)/urdf/titania.urdf.xacro" />
-    <xacro:titania_camera camera_name="$(arg camera_name)" en_mesh="$(arg en_mesh)" en_imu="$(arg en_imu)"/>
+    <!-- collision disabled in camera to avoid robot getting stuck in the floor at startup -->
+    <xacro:titania_camera camera_name="$(arg camera_name)" en_collision="true" en_mesh="$(arg en_mesh)" en_imu="$(arg en_imu)"/>
     <xacro:include filename="$(find i3dr_kinova)/urdf/interfacing_plate.urdf.xacro" />
-    <xacro:interfacing_plate />
-    <xacro:include filename="$(find i3dr_kinova)/urdf/$(arg arm_name).xacro" />
+    <!-- collision disabled in camera to avoid robot getting stuck in the floor at startup -->
+    <xacro:interfacing_plate en_collision="true" />
+    <xacro:include filename="$(find kinova_description)/urdf/$(arg arm_name).xacro" />
     <link name="root" />
     <xacro:j2s7s000 base_parent="root"/>

File: urdf/interfacing_plate.urdf.xacro (robot description, xacro)
@@ -5,11 +5,11 @@
 -->
 <robot xmlns:xacro="http://wiki.ros.org/xacro">
-    <xacro:macro name="interfacing_plate">
+    <xacro:macro name="interfacing_plate" params="en_collision:=true">
     <xacro:property name="mesh_file" value="package://i3dr_kinova/mesh/interfacing_plate_kinova.stl"/>
     <xacro:property name="mesh_offset_xyz" value="0 0 1.277"/>
     <xacro:property name="mesh_offset_rpy" value="0 ${pi} ${pi/2}"/>
-    <xacro:property name="mesh_height" value="0.059"/>
+    <xacro:property name="mesh_height" value="0.075"/>
     <xacro:property name="mesh_width" value="0.126"/>
-    <xacro:property name="mesh_length" value="0.0655"/>
+    <xacro:property name="mesh_length" value="0.075"/>
     <material name="interfacing_plate_darkgrey">
         <color rgba= "0.1 0.1 0.1 1.0"/>
@@ -22,9 +22,11 @@
             <inertia ixx="0" ixy="0" ixz="0" iyy="0" iyz="0" izz="0"/>
         </inertial>
-        <!--<collision name="interfacing_plate_collision">
-            <geometry>
-                <box size="${mesh_length} ${mesh_width} ${mesh_height}"/>
-            </geometry>
-        </collision>-->
+        <xacro:if value="${(en_collision == 'true')}">
+            <collision name="interfacing_plate_collision">
+                <geometry>
+                    <box size="${mesh_length} ${mesh_width} ${mesh_height}"/>
+                </geometry>
+            </collision>
+        </xacro:if>
         <visual>
             <origin xyz="${mesh_offset_xyz}" rpy="${mesh_offset_rpy}"/>
