Commit message: add titania kinova moveit config

File: i3dr_kinova_control/urdf/i3dr_titania_kinova_standalone.urdf.xacro (robot description, xacro)
@@ -3,5 +3,5 @@
 Copyright (c) 2019, I3D Robotics Ltd.
 -->
-<robot name="i3dr_titania_ur10"
+<robot name="i3dr_titania_kinova"
     xmlns:xacro="http://wiki.ros.org/xacro">
     <xacro:arg name="en_imu" default="false"/>
@@ -11,8 +11,8 @@
     <xacro:include filename="$(find i3dr_titania)/urdf/titania.urdf.xacro" />
     <!-- collision disabled in camera to avoid robot getting stuck in the floor at startup -->
-    <xacro:titania_camera camera_name="$(arg camera_name)" en_collision="true" en_mesh="$(arg en_mesh)" en_imu="$(arg en_imu)"/>
-    <xacro:include filename="$(find i3dr_kinova)/urdf/interfacing_plate.urdf.xacro" />
+    <xacro:titania_camera camera_name="$(arg camera_name)" en_collision="false" en_mesh="$(arg en_mesh)" en_imu="$(arg en_imu)"/>
+    <xacro:include filename="$(find i3dr_kinova_control)/urdf/interfacing_plate.urdf.xacro" />
     <!-- collision disabled in camera to avoid robot getting stuck in the floor at startup -->
-    <xacro:interfacing_plate en_collision="true" />
+    <xacro:interfacing_plate en_collision="false" />
     <xacro:include filename="$(find kinova_description)/urdf/$(arg arm_name).xacro" />
     <link name="root" />

File: i3dr_kinova_control/urdf/interfacing_plate.urdf.xacro (robot description, xacro)
@@ -6,5 +6,5 @@
 <robot xmlns:xacro="http://wiki.ros.org/xacro">
     <xacro:macro name="interfacing_plate" params="en_collision:=true">
-    <xacro:property name="mesh_file" value="package://i3dr_kinova/mesh/interfacing_plate_kinova.stl"/>
+    <xacro:property name="mesh_file" value="package://i3dr_kinova_control/mesh/interfacing_plate_kinova.stl"/>
     <xacro:property name="mesh_offset_xyz" value="0 0 1.277"/>
     <xacro:property name="mesh_offset_rpy" value="0 ${pi} ${pi/2}"/>
