Commit message: rotate interface plate to match real world

File: i3dr_kinova_control/urdf/i3dr_titania_kinova_gen3_standalone.urdf.xacro (robot description, xacro)
@@ -25,5 +25,5 @@
         <parent link="end_effector_link" />
         <child link = "interfacing_plate_base_link" />
-        <origin xyz="0 0 0" rpy="0 0 0" />
+        <origin xyz="0 0 0" rpy="0 0 1.570796327" />
     </joint>
     <joint name="interface_titania_joint" type="fixed">
